Commit message: Colors

File: install/difrobot_description/share/difrobot_description/urdf/difrobot.urdf.xacro (robot description, xacro)
@@ -4,5 +4,5 @@
   <xacro:include filename="$(find difrobot_description)/urdf/difrobot_gazebo.xacro" />
   <xacro:include filename="$(find difrobot_description)/urdf/difrobot_ros2_control.xacro" />
-    <!-- Definir Materiales -->
+  <!-- Definir Materiales -->
   <material name="red">
     <color rgba="1 0 0 1"/>
@@ -14,4 +14,11 @@
     <color rgba="0 1 0 1"/>
   </material>
+  <material name="yellow">
+    <color rgba="1 1 0 1"/> <!-- Amarillo opaco -->
+  </material>
+  <material name="purple">
+    <color rgba="0.5 0 0.5 1"/> <!-- Púrpura opaco -->
+  </material>
+  <!-- Enlaces y Joints -->
   <link name="base_footprint"/>
   <link name="base_link">
@@ -55,5 +62,12 @@
         <mesh filename="package://difrobot_description/meshes/wheel_right_link.STL" />
       </geometry>
-      <material name="green"/>  <!-- Asignar color azul -->
+      <material name="green"/>  <!-- Asignar color verde -->
+      <gazebo>
+        <material>
+          <ambient>0 0 1 1</ambient>
+          <diffuse>0 0 1 1</diffuse>
+          <specular>0 0 0 1</specular>
+        </material>
+      </gazebo>
     </visual>
     <collision>
@@ -70,6 +84,5 @@
     <axis xyz="0 1 0" />
   </joint>
-  <link
-    name="wheel_left_link">
+  <link name="wheel_left_link">
     <inertial>
       <origin xyz="0 0.014 0" rpy="0 0 0" />
@@ -84,5 +97,5 @@
         <mesh filename="package://difrobot_description/meshes/wheel_left_link.STL" />
       </geometry>
-      <material name="green"/>  <!-- Asignar color azul -->
+      <material name="green"/>  <!-- Asignar color verde -->
     </visual>
     <collision>
@@ -112,4 +125,5 @@
         <mesh filename="package://difrobot_description/meshes/caster_front_link.STL" />
       </geometry>
+      <material name="yellow"/>  <!-- Asignar color amarillo -->
     </visual>
     <collision>
@@ -139,4 +153,5 @@
         <mesh filename="package://difrobot_description/meshes/caster_rear_link.STL" />
       </geometry>
+      <material name="purple"/>  <!-- Asignar color púrpura -->
     </visual>
     <collision>

File: install/difrobot_description/share/difrobot_description/urdf/difrobot_gazebo.xacro (robot description, xacro)
@@ -1,4 +1,19 @@
 <?xml version="1.0"?>
 <robot name="difrobot" xmlns:xacro="http://ros.org/wiki/xacro">
+  <gazebo reference = "base_link">
+    <material>Gazebo/Blue</material>
+  </gazebo>
+  <gazebo reference = "wheel_left_link">
+    <material>Gazebo/Green</material>
+  </gazebo>
+  <gazebo reference = "wheel_right_link">
+    <material>Gazebo/Green</material>
+  </gazebo>
+  <gazebo reference = "caster_front_link">
+    <material>Gazebo/Yellow</material>
+  </gazebo>
+  <gazebo reference = "caster_rear_link">
+    <material>Gazebo/Purple</material>
+  </gazebo>
 <transmission name = "wheel_right_transmission">
   <plugin>transmission_interface/SimpleTransmission</plugin>
